Commit message: feat: add proper URDF from CAD model (robotV2)

File: robotV2.urdf (robot description, URDF)
Before this commit: robot my_agv_robot, 6 links, 5 joints
Links:
- removed link laser_frame
- added link lidar_link; collision cylinder length=0.04 radius=0.035; visual cylinder length=0.04 radius=0.035
Joints:
- joint lidar_joint: child laser_frame -> lidar_link
