Commit message: fix: TF timestamp offset -100ms, AMCL auto-init, costmap transform_tolerance 5.0s, URDF comments

File: test.urdf (robot description, URDF)
Before this commit: robot my_agv_robot, 6 links, 5 joints
Joints:
- joint caster_joint: origin xyz=-0.135 0 -0.0175 rpy=0 0 0 -> xyz=0.135 0 -0.0175 rpy=0 0 0
- joint left_wheel_joint: origin xyz=0.02 0.1 0 rpy=0 0 0 -> xyz=-0.02 0.1 0 rpy=0 0 0
- joint lidar_joint: origin xyz=-0.05 0 0.17 rpy=0 0 0 -> xyz=0.05 0 0.17 rpy=0 0 0
- joint right_wheel_joint: origin xyz=0.02 -0.1 0 rpy=0 0 0 -> xyz=-0.02 -0.1 0 rpy=0 0 0
